Commit message: Add new files and update existing package components

File: description/robot_core.xacro (robot description, xacro)
@@ -21,5 +21,10 @@
     </material>
     <!-- BASE LINK (Empty reference frame) -->
-    <link name="base_link">
+    <joint name="base_footprint_joint" type="fixed">
+        <parent link="base_link"/>
+        <child link="base_footprint"/>
+        <origin xyz="0 0 0" rpy="0 0 0"/>
+    </joint>
+    <link name="base_footprint">
     </link>
     <!-- CHASSIS LINK -->
